File: SARA_BreakOut/_saved_SARA_BreakOut.sch (KiCad schematic (older format))
At the start: 61 parts, among them J1 USB_B, J12 Batt_conn, J13 3v8 tp, J14 1v8 tp, J15 Mechanical_slot, J16 1,2:Vusb_bat/3,4:Vxplain, J2 Conn_02x10_Odd_Even, J3 cur_tp, J4 txd, J5 rxd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

Commit message: final schem, before starting pcb
Parts:
- J12: footprint Pin_Headers:Pin_Header_Straight_1x02_Pitch2.54mm -> Pin_Headers:Pin_Header_Angled_1x02_Pitch2.54mm
Changed lines of the file:
@@
 F 0 "J12" H 6650 6950 50  0000 C CNN
 F 1 "Batt_conn" H 6650 6650 50  0000 C CNN
-F 2 "Pin_Headers:Pin_Header_Straight_1x02_Pitch2.54mm" H 6650 6850 50  0001 C CNN
+F 2 "Pin_Headers:Pin_Header_Angled_1x02_Pitch2.54mm" H 6650 6850 50  0001 C CNN
 F 3 "" H 6650 6850 50  0001 C CNN
 	1    6650 6850
