File: SARA_BreakOut/Batt_and_LEDs.sch (KiCad schematic (older format))
At the start: 21 parts, among them J17 priority1_1,2:on/3,4:off, J18 priority2_1,2:on/3,4:off, J8 EXT_BATT, J9 conn_to_board

Commit message: first finish of pcb
Parts:
- removed D10: network, LEDs:LED_1206_HandSoldering, symbol LED
- removed D11: mod_status, LEDs:LED_1206_HandSoldering, symbol LED
- removed D12: sim, LEDs:LED_1206_HandSoldering, symbol LED
- removed D6: sara_tx, LEDs:LED_1206_HandSoldering, symbol LED
- removed D7: sara_rx, LEDs:LED_1206_HandSoldering, symbol LED
- removed D8: pwr_on, LEDs:LED_1206_HandSoldering, symbol LED
- removed D9: v_int, LEDs:LED_1206_HandSoldering, symbol LED
- removed J17: priority1_1,2:on/3,4:off, Pin_Headers:Pin_Header_Straight_1x02_Pitch2.54mm, symbol Conn_02x02_Odd_Even
- removed J18: priority2_1,2:on/3,4:off, Pin_Headers:Pin_Header_Straight_1x02_Pitch2.54mm, symbol Conn_02x02_Odd_Even
- removed R10, R11, R12, R13, R14, R15, R9: 2k, Resistors_SMD:R_1206_HandSoldering, symbol R
- BT1: footprint (none) -> Battery_Holders:Keystone_3008_1x2450-CoinCell
- C27: footprint (none) -> Capacitors_Tantalum_SMD:CP_Tantalum_Case-E_EIA-7260-38_Hand
- C28: footprint (none) -> Capacitors_SMD:C_1206_HandSoldering
- J8, J9: footprint (none) -> Pin_Headers:Pin_Header_Angled_1x02_Pitch2.54mm
Connections:
- net labels removed: GND, gpio1, gpio5, gpio6, pwr_on, rxd, txd, v_int
- wire segments 44 -> 16
- no-connect marks 4 -> 0
